File: kicad/PCB_v2/orbigator.kicad_pcb (KiCad board)
At the start: 2 copper layers, 70 x 50.5 mm, 52 parts, among them J1 Conn_01x01, J10 Conn_01x01, J11 Conn_01x01, J12 Conn_01x01, J13 Conn_01x01, J14 Conn_01x01, J15 Conn_01x01, J16 Conn_01x01, J17 Conn_01x01, J18 Conn_01x01, J19 Conn_01x01, J2 Conn_01x01, J20 Conn_01x01, J21 Conn_01x01, J22 Conn_01x01, J23 Conn_01x01, J24 Conn_01x01, J25 Conn_01x01, J26 Conn_01x01, J27 Barrel_Jack_Switch, J3 Conn_01x01, J31 Conn_01x01, J32 Conn_01x01, J33 Conn_01x01, J34 Conn_01x01, J35 Conn_01x01, J36 Conn_01x01, J37 Conn_01x01, J4 Conn_01x01, J5 Conn_01x01, J6 Conn_01x01, J7 Conn_01x01, J8 Conn_01x01, J9 Conn_01x01, M1 DYNAMIXEL_1, M2 DYNAMIXEL_2, Q1 DMG2305UX, U1 Pico_2, U2 74LS126, U3 DC_polarity, U4 DS3232M

Commit message: v2 PCB WiP
Parts:
- removed J31, J33: Conn_01x01, orbigator:PinHeader_1x01_P2.54mm_Vertical
- removed RTC1: DS3232, orbigator:DS3232_RTC_vert
- BT1: footprint Battery:BatteryHolder_LINX_BAT-HLD-012-SMT -> orbigator:BatteryHolder_LINX_BAT-HLD-012-SMT; moved to B.Cu
- C1, C2: footprint Capacitor_SMD:C_0805_2012Metric_Pad1.18x1.45mm_HandSolder -> orbigator:C_0805_2012Metric_Pad1.18x1.45mm_HandSolder
- D1: footprint PCM_Diode_SMD_AKL:D_SMA -> orbigator:D_SMA
- Q1: footprint PCM_Package_TO_SOT_SMD_AKL:SOT-23 -> orbigator:SOT-23
- R1, R2, R3, R4, R5: footprint Resistor_SMD:R_0805_2012Metric_Pad1.20x1.40mm_HandSolder -> orbigator:R_0805_2012Metric_Pad1.20x1.40mm_HandSolder
- U2: footprint Package_SO:SOIC-14_3.9x8.7mm_P1.27mm -> orbigator:SOIC-14_3.9x8.7mm_P1.27mm
- U4: footprint Package_SO:SOIC-8_3.9x4.9mm_P1.27mm -> orbigator:SOIC-8_3.9x4.9mm_P1.27mm
- moved BT1 103.3 mm to (48.6, 125.5), turned to 180 degrees
- moved U4 65.0 mm to (78.8, 122.4)
- moved C2 65.0 mm to (83.7, 124.1)
- moved C1 64.3 mm to (73.8, 122.8), turned to -90 degrees
- moved R5 59.9 mm to (78.8, 126.2)
- moved R4 58.9 mm to (78.8, 118.6), turned to 180 degrees
- moved U2 17.2 mm to (97.9, 122.4), turned to 0 degrees
- moved R3 13.0 mm to (105.2, 119.0), turned to 0 degrees
- moved U3 13.0 mm to (131.5, 118.6), turned to 180 degrees
- moved R1 12.7 mm to (105.2, 124.0), turned to 0 degrees
- moved R2 12.4 mm to (105.2, 121.5), turned to 0 degrees
- moved M1 11.8 mm to (110.6, 127.2)
- moved M2 11.8 mm to (110.6, 119.6)
- moved J20 11.2 mm to (98.3, 116.5)
- moved D1 6.34 mm to (121.0, 125.2)
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Connections:
- J25 pad 1: /5V0 -> /V_BUS
Routing:
- net /GND: track 0.00 -> 301.4 mm, vias 0 -> 7
- net /3V3: track 0.00 -> 125.6 mm, vias 0 -> 3
- net /SDA: track 0.00 -> 94.9 mm, vias 0 -> 3
- net /SCL: track 0.00 -> 92.4 mm, vias 0 -> 3
- net /V_SYS: track 0.00 -> 71.3 mm, vias 0 -> 1
- net /V_BUS: track 0.00 -> 68.0 mm, vias 0 -> 1
- net /MOT_DAT: track 0.00 -> 62.5 mm
- net /ENC_SW: track 0.00 -> 35.5 mm, vias 0 -> 1
- net /ENC_A: track 0.00 -> 34.0 mm, vias 0 -> 1
- net /ENC_B: track 0.00 -> 33.7 mm, vias 0 -> 1
- net /CNF_BTN: track 0.00 -> 31.9 mm, vias 0 -> 1
- net /5V0: track 0.00 -> 30.1 mm
- net /BAK_BTN: track 0.00 -> 29.3 mm, vias 0 -> 1
- net /UART_TX: track 0.00 -> 28.0 mm, vias 0 -> 2
- net /DIR: track 0.00 -> 15.7 mm
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- added copper zone on B.Cu, net /GND
